Commit message: Added new Nodes

File: src/robot/urdf/robot.urdf (robot description, URDF)
Before this commit: robot mobile_manipulator, 12 links, 11 joints
Links:
- removed link arm_base_link
- removed link base_link
- removed link elbow_link
- removed link front_left_wheel_link
- removed link front_right_wheel_link
- removed link rear_left_wheel_link
- removed link rear_right_wheel_link
- removed link shoulder_link
- removed link tool0
- removed link wrist_1_link
- removed link wrist_2_link
- removed link wrist_3_link
- added link back_left_wheel, mass 0.5; collision cylinder length=0.04 radius=0.06; visual cylinder length=0.04 radius=0.06
- added link back_right_wheel, mass 0.5; collision cylinder length=0.04 radius=0.06; visual cylinder length=0.04 radius=0.06
- added link base_rotator_link, mass 1.8; collision box size=0.1 0.1 0.18; visual box size=0.08 0.08 0.18
- added link chassis_link, mass 6.5; collision box size=0.4 0.3 0.1; collision cylinder length=0.05 radius=0.075
- added link forearm_link, mass 1.5; collision box size=0.07 0.07 0.15; visual box size=0.065 0.065 0.15
- added link front_left_wheel, mass 0.5; collision cylinder length=0.04 radius=0.06; visual cylinder length=0.04 radius=0.06
- added link front_right_wheel, mass 0.5; collision cylinder length=0.04 radius=0.06; visual cylinder length=0.04 radius=0.06
- added link gripper1_link, mass 0.1; collision box size=0.01 0.01 0.01; collision box size=0.01 0.01 0.05
- added link gripper2_link, mass 0.1; collision box size=0.01 0.01 0.01; collision box size=0.01 0.01 0.05
- added link upper_arm_link, mass 1.8; collision box size=0.08 0.08 0.2; visual box size=0.07 0.07 0.2
- added link wrist_pitch_link, mass 0.8; collision box size=0.06 0.06 0.18; visual box size=0.055 0.055 0.18
- added link wrist_roll_link, mass 0.4; collision box size=0.08 0.06 0.06; visual box size=0.05 0.045 0.04
Joints:
- removed joint arm_joint_1
- removed joint arm_joint_2
- removed joint arm_joint_3
- removed joint arm_joint_4
- removed joint arm_joint_5
- removed joint arm_joint_6
- removed joint front_left_wheel
- removed joint front_right_wheel
- removed joint rear_left_wheel
- removed joint rear_right_wheel
- removed joint tool_joint
- added joint back_left_wheel_joint: type continuous, parent chassis_link, child back_left_wheel, origin xyz=-0.15 0.18 -0.05 rpy=-1.5708 0 0, axis 0 0 1
- added joint back_right_wheel_joint: type continuous, parent chassis_link, child back_right_wheel, origin xyz=-0.15 -0.18 -0.05 rpy=-1.5708 0 0, axis 0 0 1
- added joint base_yaw_joint: type revolute, parent chassis_link, child base_rotator_link, origin xyz=0 0 0.10 rpy=0 0 0, axis 0 0 1, limit lower=-3.14 upper=3.14 effort=5.0 velocity=1.0
- added joint elbow_joint: type revolute, parent upper_arm_link, child forearm_link, origin xyz=0 0 0.2 rpy=0 0 0, axis 0 1 0, limit lower=0 upper=1.5708 effort=100 velocity=1.0
- added joint front_left_wheel_joint: type continuous, parent chassis_link, child front_left_wheel, origin xyz=0.15 0.18 -0.05 rpy=-1.5708 0 0, axis 0 0 1
- added joint front_right_wheel_joint: type continuous, parent chassis_link, child front_right_wheel, origin xyz=0.15 -0.18 -0.05 rpy=-1.5708 0 0, axis 0 0 1
- added joint gripper2_joint: type prismatic, parent wrist_roll_link, child gripper2_link, origin xyz=0 0 0.05 rpy=0 0 0, axis 0 -1 0, limit lower=0 upper=0.03 effort=10 velocity=0.05, mimic joint=gripper_joint multiplier=1.0 offset=0
- added joint gripper_joint: type prismatic, parent wrist_roll_link, child gripper1_link, origin xyz=0 0 0.05 rpy=0 0 0, axis 0 1 0, limit lower=0 upper=0.03 effort=10 velocity=0.05
- added joint shoulder_joint: type revolute, parent base_rotator_link, child upper_arm_link, origin xyz=0 0 0.18 rpy=0 0 0, axis 0 1 0, limit lower=-1.5708 upper=1.5708 effort=100 velocity=1.0
- added joint wrist_pitch_joint: type revolute, parent forearm_link, child wrist_pitch_link, origin xyz=0 0 0.15 rpy=0 0 0, axis 0 1 0, limit lower=-1.5708 upper=1.5708 effort=100 velocity=1.0
- added joint wrist_roll_joint: type revolute, parent wrist_pitch_link, child wrist_roll_link, origin xyz=0 0 0.1775 rpy=0 0 0, axis 0 0 1, limit lower=-3.14 upper=3.14 effort=100 velocity=1.0
